Commit message: updates to rassor xacro

File: packages/simulation/ezrassor_sim_description/urdf/ezrassor.xacro (robot description, xacro)
@@ -24,5 +24,5 @@
       <origin xyz="0 0 0" rpy=" 0 0 0"/>
       <geometry>
-        <base_unit/>
+        <xacro:base_unit/>
       </geometry>
     </collision>
@@ -30,5 +30,5 @@
       <origin xyz="0 0 0" rpy=" 0 0 0"/>
       <geometry>
-        <base_unit/>
+        <xacro:base_unit/>
       </geometry>
     </visual>
@@ -38,5 +38,5 @@
       <origin xyz="0 0 0" rpy="0 0 0"/>
       <geometry>
-        <robot_wheel />
+        <xacro:robot_wheel />
       </geometry>
       <surface>
@@ -56,5 +56,5 @@
       <origin xyz="0 0 0" rpy="0 0 0"/>
       <geometry>
-        <robot_wheel />
+        <xacro:robot_wheel />
       </geometry>
     </visual>
@@ -62,5 +62,5 @@
       <origin xyz="0 0 0" rpy="0 0 0" />
       <mass value="5"/>
-      <cylinder_inertia m="5" r="0.18" h="0.2"/>
+      <xacro:cylinder_inertia m="5" r="0.18" h="0.2"/>
     </inertial>
   </link>
@@ -69,5 +69,5 @@
       <origin xyz="0 0 0" rpy="0 0 3.14159"/>
       <geometry>
-        <robot_wheel />
+        <xacro:robot_wheel />
       </geometry>
       <surface>
@@ -81,11 +81,11 @@
       <origin xyz="0 0 0" rpy="0 0 3.14159"/>
       <geometry>
-        <robot_wheel />
-      </geometry>
-    </visual>
-    <inertial>
-      <origin xyz="0 0 0" rpy="0 0 3.14159"/>
-      <mass value="5"/>
-      <cylinder_inertia m="5" r="0.18" h="0.2"/>
+        <xacro:robot_wheel />
+      </geometry>
+    </visual>
+    <inertial>
+      <origin xyz="0 0 0" rpy="0 0 3.14159"/>
+      <mass value="5"/>
+      <xacro:cylinder_inertia m="5" r="0.18" h="0.2"/>
     </inertial>
   </link>
@@ -94,5 +94,5 @@
       <origin xyz="0 0 0" rpy="0 0 0"/>
       <geometry>
-        <robot_wheel />
+        <xacro:robot_wheel />
       </geometry>
         <surface>
@@ -106,11 +106,11 @@
       <origin xyz="0 0 0" rpy="0 0 0"/>
       <geometry>
-        <robot_wheel />
-      </geometry>
-    </visual>
-    <inertial>
-      <origin xyz="0 0 0" rpy="0 0 0"/>
-      <mass value="5"/>
-      <cylinder_inertia m="5" r="0.18" h="0.2"/>
+        <xacro:robot_wheel />
+      </geometry>
+    </visual>
+    <inertial>
+      <origin xyz="0 0 0" rpy="0 0 0"/>
+      <mass value="5"/>
+      <xacro:cylinder_inertia m="5" r="0.18" h="0.2"/>
     </inertial>
   </link>
@@ -119,5 +119,5 @@
       <origin xyz="0 0 0" rpy="0 0 3.14159"/>
       <geometry>
-        <robot_wheel />
+        <xacro:robot_wheel />
       </geometry>
       <surface>
@@ -131,11 +131,11 @@
       <origin xyz="0 0 0" rpy="0 0 3.14159"/>
       <geometry>
-        <robot_wheel />
-      </geometry>
-    </visual>
-    <inertial>
-      <origin xyz="0 0 0" rpy="0 0 3.14159"/>
-      <mass value="5"/>
-      <cylinder_inertia m="5" r="0.18" h="0.2"/>
+        <xacro:robot_wheel />
+      </geometry>
+    </visual>
+    <inertial>
+      <origin xyz="0 0 0" rpy="0 0 3.14159"/>
+      <mass value="5"/>
+      <xacro:cylinder_inertia m="5" r="0.18" h="0.2"/>
     </inertial>
   </link>
@@ -144,5 +144,5 @@
       <origin xyz="0 0 0" rpy="0 0 0"/>
       <geometry>
-        <drum_arm />
+        <xacro:drum_arm />
       </geometry>
     </collision>
@@ -150,11 +150,11 @@
       <origin xyz="0 0 0" rpy="0 0 0" />
       <geometry>
-        <drum_arm />
-      </geometry>
-    </visual>
-    <inertial>
-      <origin xyz="0 0 0" rpy="0 0 0"/>
-      <mass value="5"/>
-      <cylinder_inertia m="5" r="0.05" h="0.3"/>
+        <xacro:drum_arm />
+      </geometry>
+    </visual>
+    <inertial>
+      <origin xyz="0 0 0" rpy="0 0 0"/>
+      <mass value="5"/>
+      <xacro:cylinder_inertia m="5" r="0.05" h="0.3"/>
     </inertial>
   </link>
@@ -163,5 +163,5 @@
       <origin xyz="0 0 0" rpy="3.1415 0 3.1415"/>
       <geometry>
-        <drum_arm />
+        <xacro:drum_arm />
       </geometry>
     </collision>
@@ -169,5 +169,5 @@
       <origin xyz="0 0 0" rpy="3.1415 0 3.1415"/>
       <geometry>
-        <drum_arm />
+        <xacro:drum_arm />
       </geometry>
     </visual>
@@ -198,11 +198,11 @@
       <origin xyz="0 0 0" rpy="0 0 0"/>
       <geometry>
-        <robot_arm_drum />
-      </geometry>
-    </visual>
-    <inertial>
-      <origin xyz="0 0 0" rpy="0 0 0"/>
-      <mass value="5"/>
-      <cylinder_inertia m="5" r="0.1839" h="1.0"/>
+        <xacro:robot_arm_drum />
+      </geometry>
+    </visual>
+    <inertial>
+      <origin xyz="0 0 0" rpy="0 0 0"/>
+      <mass value="5"/>
+      <xacro:cylinder_inertia m="5" r="0.1839" h="1.0"/>
     </inertial>
   </link>
@@ -223,11 +223,11 @@
       <origin xyz="0 0 0" rpy="3.1415 0 3.14159"/>
       <geometry>
-        <robot_arm_drum />
-      </geometry>
-    </visual>
-    <inertial>
-      <origin xyz="0 0 0" rpy="0 0 3.14159"/>
-      <mass value="5"/>
-      <cylinder_inertia m="5" r="0.1839" h="1.0"/>
+        <xacro:robot_arm_drum />
+      </geometry>
+    </visual>
+    <inertial>
+      <origin xyz="0 0 0" rpy="0 0 3.14159"/>
+      <mass value="5"/>
+      <xacro:cylinder_inertia m="5" r="0.1839" h="1.0"/>
     </inertial>
   </link>
